File: st-breakout/st-breakout.sch (KiCad schematic (older format))
At the start: 12 parts

Commit message: Change MCU model, Fill schematic and footprints
Parts:
- removed C? (x2): 100n, symbol Device:C_Small
- removed C? (x2): 10p, symbol Device:C_Small
- removed L?: 39n, symbol Device:L
- removed R?: 47, symbol Device:R
- removed U?: STM32F103C8T6, Package_QFP:LQFP-48_7x7mm_P0.5mm, symbol MCU_ST_STM32F1:STM32F103C8Tx
- removed Y?: 16MHz, symbol Device:Crystal_GND24
- added C1, C6: 100n, Capacitor_SMD:C_0402_1005Metric, symbol Device:C_Small
- added C10: 1u, Capacitor_SMD:C_0402_1005Metric, symbol Device:C_Small
- added C11, C12: 30p, Capacitor_SMD:C_0402_1005Metric, symbol Device:C_Small
- added C2: 10u, Capacitor_SMD:C_0603_1608Metric, symbol Device:C_Small
- added C8, C9: 22u, Capacitor_SMD:C_0805_2012Metric, symbol Device:C_Small
- added D1: RED USER_LED, LED_SMD:LED_0603_1608Metric, symbol Device:LED
- added D2: GREEN STATUS_LED, LED_SMD:LED_0603_1608Metric, symbol Device:LED_Small
- added FB1: 220R, Inductor_SMD:L_0603_1608Metric, symbol Device:Ferrite_Bead
- added J1: SPI, Connector_PinHeader_2.54mm:PinHeader_1x05_P2.54mm_Vertical, symbol Connector_Generic:Conn_01x05
- added J2: SWD, Connector_PinHeader_2.54mm:PinHeader_1x05_P2.54mm_Vertical, symbol Connector_Generic:Conn_01x05
- added J3: USB_C_Receptacle_USB2.0, symbol Connector:USB_C_Receptacle_USB2.0
- added J4: USART, Connector_PinSocket_2.54mm:PinSocket_1x04_P2.54mm_Vertical, symbol Connector_Generic:Conn_01x04
- added L1: 3u9, Inductor_SMD:L_0603_1608Metric, symbol Device:L_Small
- added R1: 619R, Resistor_SMD:R_0402_1005Metric, symbol Device:R
- added R2: 619R, Resistor_SMD:R_0402_1005Metric, symbol Device:R_Small
- added R3: 1k5, Resistor_SMD:R_0402_1005Metric, symbol Device:R
- added R4: 22R, Resistor_SMD:R_0402_1005Metric, symbol Device:R_Small
- added R5: 47R, Resistor_SMD:R_0402_1005Metric, symbol Device:R
- added R6, R7: 5k1, Resistor_SMD:R_0402_1005Metric, symbol Device:R_Small
- added SW1: SW_SPDT, Button_Switch_SMD:SW_SPDT_PCM12, symbol Switch:SW_SPDT
- added U1: AP63203WU, Package_TO_SOT_SMD:TSOT-23-6, symbol Regulator_Switching:AP63203WU
- added U2: STM32F070F6P6TR, Package_SO:TSSOP-20_4.4x6.5mm_P0.65mm, symbol MCU_ST_STM32F0:STM32F070F6Px
- added Y1: 16 MHz, Crystal:Crystal_SMD_HC49-SD, symbol Device:Crystal
- C3, C5: renamed from C?; footprint (none) -> Capacitor_SMD:C_0603_1608Metric
- C4, C7: renamed from C?; footprint (none) -> Capacitor_SMD:C_0402_1005Metric
Connections:
- net labels added: BOOT, NRST, SPI_MISO, SPI_MOSI, SPI_SCK, VBUS
- net labels removed: I2C_SCL, I2C_SDA, RST, STATUS_LED, SWO
- wire segments 36 -> 70
- no-connect marks 25 -> 6
Other:
- note added: "3.3V 2A Buck Converter"
- note added: "Analog Filtering"
- note added: "Boot Mode Switch"
- note added: "Crystal Oscillator"
- note added: "STM32F070F6P6TR"
- note added: "USB-C\n"
- note removed: "STM32F103C8T6 MCU"
- moved on the sheet: C3, C4, C5, C7
