File: st-breakout/st-breakout.kicad_sch (KiCad schematic)
At the start: 35 parts, among them J1 SPI, J2 SWD, J3 USB4085-GF-A_REVB, J4 USART, SW1 SW_SPDT, U1 AP63203WU, U2 STM32F070F6Px, Y1 16 MHz

Commit message: routing and gerber
Parts:
- removed J3: USB4085-GF-A_REVB, USB4085-GF-A:GCT_USB4085-GF-A_REVB, symbol USB4085-GF-A_REVB:USB4085-GF-A_REVB
- added J5: USB4105-GF-A-060, USB4105-GF-A-060:GCT_USB4105-GF-A-060, symbol USB4105-GF-A-060:USB4105-GF-A-060
Connections:
- net GND: now also R5.1, R6.1, J5.A1_B12 (GND), J5.B1_A12 (GND); no longer R5.2, R6.2
- net USART_RX: now also J4.2 (Pin_2); no longer J4.3 (Pin_3)
- net USART_TX: now also J4.3 (Pin_3); no longer J4.2 (Pin_2)
- net USB_D+: now also J5.A6 (DP1), J5.B6 (DP2)
- net USB_D-: now also J5.A7 (DN1), J5.B7 (DN2)
- net VBUS: now also J5.A4_B9 (VBUS), J5.B4_A9 (VBUS)
- new net: J5.A5 (CC1), R5.2
- new net: J5.B5 (CC2), R6.2
- new net: J5.S1 (SHELL_GND), J5.S2 (SHELL_GND), J5.S3 (SHELL_GND), J5.S4 (SHELL_GND)
Other:
- note added: "M2"
- moved on the sheet: H2, H3, H4, R5, R6
